File: pcb/eagle/waterlezer.brd (EAGLE design)
At the start: 30.5 x 49.2 mm, 9 parts, among them IC1 OP-AMP

Commit message: cleanup
Parts:
- IC1: value OP-AMP -> LMV358P
Changed lines of the file:
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@@
 <attribute name="VALUE" x="19.16898125" y="12.34" size="1.27373125" layer="28" ratio="10" rot="MR270" align="top-left"/>
 </element>
-<element name="IC1" library="SparkFun-IC-Amplifiers" library_urn="urn:adsk.eagle:library:520" package="DIP08" package3d_urn="urn:adsk.eagle:package:38666/1" value="OP-AMP" x="15.24" y="36.83" smashed="yes" rot="R180">
+<element name="IC1" library="SparkFun-IC-Amplifiers" library_urn="urn:adsk.eagle:library:520" package="DIP08" package3d_urn="urn:adsk.eagle:package:38666/1" value="LMV358P" x="15.24" y="36.83" smashed="yes" rot="R180">
 <attribute name="NAME" x="20.955" y="36.83" size="0.6096" layer="25" font="vector" ratio="20" rot="R270" align="bottom-center"/>
 <attribute name="PROD_ID" value="NA-XXXXX" x="15.24" y="36.83" size="1.778" layer="27" rot="R180" display="off"/>
